File: Board/LoraSensor/LoraSensor.kicad_pcb (KiCad board)
At the start: 2 copper layers, 124.2 x 30.5 mm, 36 parts, among them J1 Conn_01x02_Socket, J2 USB_B_Micro, J4 CapSense, J5 Conn_01x03_Socket, J6 Conn_01x03_Pin, Q1 MMBT3906, U1 TPS7A2633DRVR, U2 SHTC3, U3 HT-CT62

Commit message: PCB V1.1
Parts:
- removed R4: 10k, Resistor_SMD:R_1206_3216Metric
- removed TP1: SENSE, TestPoint:TestPoint_Pad_D1.0mm
- removed TP2: PWM, TestPoint:TestPoint_Pad_D1.0mm
- removed TP3: Lora, TestPoint:TestPoint_THTPad_D2.0mm_Drill1.0mm
- added SW1: SW_Push, Custom:smd-tactile, F.Cu at (184.1, 87.2)
- moved AE1 20.9 mm to (148.7, 82.4), turned to 180 degrees
- moved R9 20.1 mm to (174.2, 80.9)
- moved JP1 14.7 mm to (174.2, 86.5), turned to 90 degrees
- moved C6 12.3 mm to (171.8, 85.0), turned to 90 degrees
- moved C7 11.7 mm to (178.8, 75.5), turned to -90 degrees
- moved U2 11.4 mm to (176.1, 75.5)
- moved D1 9.20 mm to (186.2, 62.0)
- moved R2 7.75 mm to (179.3, 85.9)
- moved R1 7.62 mm to (179.3, 80.9)
- moved AE2 5.61 mm to (147.5, 68.3)
- moved C2 4.70 mm to (179.3, 69.4), turned to 90 degrees
- moved R3 3.17 mm to (176.7, 80.9), turned to 90 degrees
- moved C1 2.97 mm to (174.2, 69.6), turned to -90 degrees
- moved C3 1.15 mm to (173.4, 63.9)
- moved U3 1.15 mm to (162.8, 73.4)
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Connections:
- J1 pad 1: GND -> VIN
- J1 pad 2: VIN -> GND
- R3 pad 1: /SCL -> /BTN
- U3 pad 10: /BATSENSE -> /SENSE
- U3 pad 14: unconnected-(U3-GPIO10-Pad14) -> /PWM
- U3 pad 19: /PWM -> /SCL
- U3 pad 8: /SCL -> /BTN
- U3 pad 9: /SENSE -> /BATSENSE
Routing:
- net +3V3: track 96.9 -> 40.5 mm, vias 2 -> 0
- net /BTN: track 0.00 -> 28.7 mm
- net Net-(AE1-FEED): track 3.66 -> 22.2 mm
- net /EN: track 11.7 -> 30.3 mm, vias 0 -> 2
- net VIN: track 13.1 -> 28.1 mm
- net Net-(AE2-FEED): track 25.6 -> 11.6 mm
- net /SDA: track 34.1 -> 21.9 mm, vias 2 -> 0
- net /PWM: track 49.7 -> 42.4 mm
- net /PWM_SENSOR: track 14.7 -> 10.1 mm
- net GND: track 52.2 -> 48.5 mm, vias 103 -> 198
- net /BATSENSE: track 27.8 -> 25.3 mm
- net /SENSE_SENSOR: track 19.3 -> 16.9 mm
- net VBUS: track 4.50 -> 6.73 mm
- net /SCL: track 23.1 -> 21.2 mm
- net Net-(JP2-A): track 1.95 -> 2.88 mm
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Other:
- outline, holes or cut-outs redrawn
- board text added: "LoRa"
- board text added: "LoraSense 1.1"
- board text removed: "LoraSense 1.0"

Commit message: Version 1.1
Parts:
- removed J5: Conn_01x03_Socket, Custom:532614003
- removed J6: Conn_01x03_Pin, Connector_PinHeader_2.54mm:PinHeader_1x03_P2.54mm_Vertical
- removed NT1, NT2: NetTie_2, NetTie:NetTie-2_SMD_Pad0.5mm
- added C8: 10n, Capacitor_SMD:C_0805_2012Metric_Pad1.18x1.45mm_HandSolder, F.Cu at (176.9, 85.2)
- added R10: 10k, Resistor_SMD:R_1206_3216Metric, F.Cu at (157.0, 61.6)
- added R4: 10k, Resistor_SMD:R_1206_3216Metric, F.Cu at (173.6, 75.6)
- moved R7 20.3 mm to (183.4, 67.1)
- moved C5 17.8 mm to (185.0, 73.2), turned to 90 degrees
- moved Q1 17.7 mm to (188.0, 68.2), turned to 0 degrees
- moved R6 15.7 mm to (182.4, 73.4)
- moved R5 14.6 mm to (183.4, 69.5), turned to 0 degrees
- moved D2 13.5 mm to (187.6, 72.5)
- moved J1 11.0 mm to (184.8, 80.9)
- moved J4 9.59 mm to (229.2, 73.5)
- moved JP1 1.15 mm to (174.3, 85.3)
- moved C1 0.40 mm to (173.9, 69.4)
- moved C2 0.40 mm to (179.0, 69.2)
- moved U1 0.40 mm to (176.5, 69.3)
Connections:
- C5 pad 1: /SENSE_SENSOR -> /SENSE
- D2 pad 1: /SENSE_SENSOR -> /SENSE
- JP2 pad 2: /GPIO9 -> /PWM
- R5 pad 1: /PWM_SENSOR -> /PWM
- R6 pad 1: /SENSE_SENSOR -> /SENSE
- R7 pad 1: /PWM_SENSOR -> /PWM
- U3 pad 14: /PWM -> unconnected-(U3-GPIO10-Pad14)
- U3 pad 15: /GPIO9 -> /PWM
Routing:
- net /CAP: track 39.8 -> 73.9 mm
- net +3V3: track 40.5 -> 61.3 mm, vias 0 -> 2
- net /SENSE_SENSOR: track 16.9 -> 0.00 mm
- net /PWM: track 42.4 -> 27.9 mm
- net /PWM_SENSOR: track 10.1 -> 0.00 mm
- net /SDA: track 21.9 -> 25.1 mm
- net VIN: track 28.1 -> 31.0 mm
- net /SENSE: track 40.4 -> 43.0 mm
- net /BATSENSE: track 25.3 -> 27.8 mm
- net /GPIO9: track 2.40 -> 0.00 mm
- net /SCL: track 21.2 -> 22.9 mm
- net /EN: track 30.3 -> 29.2 mm
- net Net-(Q1-B): track 3.25 -> 2.30 mm
- net GND: track 48.5 -> 47.9 mm, vias 198 -> 195
Other:
- board text added: "LoraSense 1.2"
- board text removed: "LoraSense 1.1"

Commit message: PCB  Version 1.2
Parts:
- moved J4 1.97 mm to (231.1, 73.7)
Other:
- outline, holes or cut-outs redrawn
Changed lines of the file:
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@@
 		)
 		(property "Value" "10n"
-			(at 0 1.68 270)
+			(at 0 1.68 -90)
 			(layer "F.Fab")
 			(effects
@@
 		)
 		(fp_text user "${REFERENCE}"
-			(at 0 0 270)
+			(at 0 0 -90)
 			(layer "F.Fab")
 			(effects
@@
 		)
 		(property "Value" "10k"
-			(at 0 1.82 360)
+			(at 0 1.82 0)
 			(layer "F.Fab")
 			(effects
@@
 		)
 		(fp_text user "${REFERENCE}"
-			(at 0 0 360)
+			(at 0 0 0)
 			(layer "F.Fab")
 			(effects
@@
 		)
 		(property "Value" "1n"
-			(at 0 1.68 270)
+			(at 0 1.68 -90)
 			(layer "F.Fab")
 			(effects
@@
 		)
 		(fp_text user "${REFERENCE}"
-			(at 0 0 270)
+			(at 0 0 -90)
 			(layer "F.Fab")
 			(effects
@@
 		(tags "SOD-323")
 		(property "Reference" "D2"
-			(at -2.413 -0.381 360)
+			(at -2.413 -0.381 0)
 			(layer "F.SilkS")
 			(effects
@@
 		)
 		(property "Value" "1N4148WS"
-			(at 0.1 1.9 270)
+			(at 0.1 1.9 -90)
 			(layer "F.Fab")
 			(effects
@@
 		)
 		(fp_text user "${REFERENCE}"
-			(at 0 -1.85 270)
+			(at 0 -1.85 -90)
 			(layer "F.Fab")
 			(effects
@@
 		(tags "resistor")
 		(property "Reference" "R9"
-			(at -0.381 -1.778 90)
+			(at -0.381 -1.524 90)
 			(layer "F.SilkS")
 			(effects
@@
 	(footprint "Custom:CapSense"
 		(layer "F.Cu")
-		(at 229.171 73.533 90)
+		(at 231.14 73.66 90)
 		(property "Reference" "J4"
 			(at 0 -0.5 90)
@@
 		(pad "1" smd oval
 			(at 0 -4 90)
-			(size 10 65)
+			(size 10 60)
 			(layers "F.Cu")
 			(net 6 "/CAP")
@@
 		(tags "SOT TO_SOT_SMD")
 		(property "Reference" "Q1"
-			(at -0.508 -2.667 360)
+			(at -0.508 -2.667 0)
 			(layer "F.SilkS")
 			(effects
@@
 		)
 		(property "Value" "MMBT3906"
-			(at 0 2.4 360)
+			(at 0 2.4 0)
 			(layer "F.Fab")
 			(effects
@@
 		)
 		(fp_text user "${REFERENCE}"
-			(at 0 0 360)
+			(at 0 0 0)
 			(layer "F.Fab")
 			(effects
@@
 	)
 	(gr_line
-		(start 197.358 66.04)
-		(end 197.358 81.28)
+		(start 200.914 66.04)
+		(end 200.914 81.28)
 		(stroke
 			(width 0.1)
@@
 	)
 	(gr_line
-		(start 197.358 66.04)
-		(end 197.358 81.28)
+		(start 200.914 66.04)
+		(end 200.914 81.28)
 		(stroke
 			(width 0.1)
@@
 	)
 	(gr_arc
-		(start 187.96 88.392)
-		(mid 187.81121 88.75121)
-		(end 187.452 88.9)
+		(start 189.23 88.392)
+		(mid 189.08121 88.75121)
+		(end 188.722 88.9)
 		(stroke
 			(width 0.1)
@@
 	)
 	(gr_arc
-		(start 188.468 63.5)
-		(mid 188.10879 63.35121)
-		(end 187.96 62.992)
+		(start 189.738 63.5)
+		(mid 189.37879 63.35121)
+		(end 189.23 62.992)
 		(stroke
 			(width 0.1)
@@
 	)
 	(gr_arc
-		(start 187.452 58.42)
-		(mid 187.81121 58.56879)
-		(end 187.96 58.928)
+		(start 188.722 58.42)
+		(mid 189.08121 58.56879)
+		(end 189.23 58.928)
 		(stroke
 			(width 0.1)
@@
 	(gr_line
 		(start 184.912 58.42)
-		(end 187.452 58.42)
+		(end 188.722 58.42)
 		(stroke
 			(width 0.1)
@@
 	)
 	(gr_line
-		(start 188.468 63.5)
+		(start 189.738 63.5)
 		(end 256.32958 63.5)
 		(stroke
@@
 	(gr_line
 		(start 256.32958 83.82)
-		(end 188.468 83.82)
+		(end 189.738 83.82)
 		(stroke
 			(width 0.1)
@@
 	)
 	(gr_line
-		(start 187.96 58.928)
-		(end 187.96 62.992)
+		(start 189.23 58.928)
+		(end 189.23 62.992)
 		(stroke
 			(width 0.1)
@@
 	)
 	(gr_line
-		(start 187.452 88.9)
+		(start 188.722 88.9)
 		(end 142.748 88.900011)
 		(stroke
@@
 	)
 	(gr_line
-		(start 187.96 84.328)
-		(end 187.96 88.392)
+		(start 189.23 84.328)
+		(end 189.23 88.392)
 		(stroke
 			(width 0.1)
@@
 	)
 	(gr_arc
-		(start 187.96 84.328)
-		(mid 188.10879 83.96879)
-		(end 188.468 83.82)
+		(start 189.23 84.328)
+		(mid 189.37879 83.96879)
+		(end 189.738 83.82)
 		(stroke
 			(width 0.1)
@@
 		(polygon
 			(pts
-				(xy 153.416 58.8676) (xy 153.416 76.2) (xy 152.146 76.2) (xy 152.146 88.8396) (xy 187.452 88.8396)
-				(xy 187.452 83.7596) (xy 256.286 83.7596) (xy 266.192 73.8536) (xy 256.286 63.9476) (xy 187.706 63.9476)
-				(xy 187.706 58.8676)
+				(xy 153.416 58.8676) (xy 153.416 76.2) (xy 152.146 76.2) (xy 152.146 88.9) (xy 188.976 88.8396)
+				(xy 188.976 83.82) (xy 256.286 83.7596) (xy 266.192 73.8536) (xy 256.286 63.9476) (xy 188.976 63.9476)
+				(xy 188.976 58.8676)
 			)
 		)
