File: Board/LoraSensor/LoraSensor.kicad_sch (KiCad schematic)
At the start: 36 parts, among them J1 Conn_01x02_Socket, J2 USB_B_Micro, J4 CapSense, J5 Conn_01x03_Socket, J6 Conn_01x03_Pin, Q1 MMBT3906, U1 TPS7A2633DRVR, U2 SHTC3, U3 HT-CT62

Commit message: PCB V1.1
Parts:
- removed R4: 10k, Resistor_SMD:R_1206_3216Metric, symbol Device:R_US
- removed TP1: SENSE, TestPoint:TestPoint_Pad_D1.0mm, symbol Connector:TestPoint
- removed TP2: PWM, TestPoint:TestPoint_Pad_D1.0mm, symbol Connector:TestPoint
- removed TP3: Lora, TestPoint:TestPoint_THTPad_D2.0mm_Drill1.0mm, symbol Connector:TestPoint
- added SW1: SW_Push, Custom:smd-tactile, symbol Switch:SW_Push
Connections:
- net BATSENSE: now also U3.9 (GPIO1); no longer U3.10 (GPIO0)
- net GND: now also J1.2 (Pin_2), SW1.2; no longer J1.1 (Pin_1)
- net PWM: now also U3.14 (GPIO10); no longer U3.19 (GPIO20_RXD)
- net SCL: now also U3.19 (GPIO20_RXD); no longer R3.1, U3.8 (GPIO2)
- net SENSE: now also U3.10 (GPIO0); no longer U3.9 (GPIO1)
- net VIN: now also J1.1 (Pin_1); no longer J1.2 (Pin_2)
- new net BTN: R3.1, SW1.1, U3.8 (GPIO2)
- no-connect marks 12 -> 11
Other:
- moved on the sheet: AE2, J1

Commit message: Version 1.1
Parts:
- removed J5: Conn_01x03_Socket, Custom:532614003, symbol Connector:Conn_01x03_Socket
- removed J6: Conn_01x03_Pin, Connector_PinHeader_2.54mm:PinHeader_1x03_P2.54mm_Vertical, symbol Connector:Conn_01x03_Pin
- removed NT1, NT2: NetTie_2, NetTie:NetTie-2_SMD_Pad0.5mm, symbol Device:NetTie_2
- added C8: 10n, Capacitor_SMD:C_0805_2012Metric_Pad1.18x1.45mm_HandSolder, symbol Device:C
- added R10, R4: 10k, Resistor_SMD:R_1206_3216Metric, symbol Device:R_US
Connections:
- net GPIO9 is gone; now on net PWM: JP2.2 (B), U3.15 (GPIO9)
- net PWM_SENSOR is gone; now on net PWM: R5.1, R7.1
- net SENSE_SENSOR is gone; now on net SENSE: C5.1, D2.1 (K), R6.1
- net +3V3: now also R10.2, R4.2
- net BATSENSE: now also C8.2
- net GND: now also C8.1
- net PWM: no longer U3.14 (GPIO10)
- net SCL: now also R4.1
- net SDA: now also R10.1
- no-connect marks 11 -> 12
Other:
- moved on the sheet: C3, C4, JP2, R3, R8, SW1

Commit message: PCB  Version 1.2
Parts:
- AE1: value Wifi -> 2450AT18A100E; Comment (none) -> Wifi
- AE2: value Lora -> ANT-868-uSP410; Comment (none) -> Lora
- C3: value 47u -> 47uF; now not fitted; now left out of the parts list
- J1: value Conn_01x02_Socket -> MOLEX PicoBlade 532614002
- J2: value USB_B_Micro -> MOLEX 473460001
- J4: now left out of the parts list
- SW1: value SW_Push -> TS-1088R-02026
Other:
- moved on the sheet: C1, C2, C5, C7, C8, D1, D2, J1, J2, Q1, R1, R2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
